File: kicad/Control/Control.kicad_pcb (KiCad board)
At the start: 2 copper layers, 75 x 75 mm, 27 parts, among them J1 Conn_01x20_Pin, J2 Conn_01x05_Pin, J3 Screw_Terminal_01x02, J4 Conn_02x05_Odd_Even, J5 Conn_02x05_Odd_Even, SW1 PRESET1, SW2 CH2_EN, SW3 PRESET2, SW4 COARSE, SW5 CH1_EN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

Commit message: Fix control connectors spacing
Parts:
- J4, J5: footprint Connector_PinHeader_2.54mm:PinHeader_2x05_P2.54mm_Vertical -> Altbutt:Connector Header 2x05
- moved H2 12.7 mm to (102.2, 112.7)
- moved J5 5.39 mm to (109.6, 119.5)
Connections:
- J4 pad 2: CH1_ADC_CS -> CH2_ADC_CS
- J4 pad 3: CH1_GND -> CH2_GND
- J4 pad 4: CH1_DAC_CS -> CH2_DAC_CS
- J4 pad 6: CH1_OUT_EN -> CH2_OUT_EN
- J5 pad 2: CH2_ADC_CS -> CH1_ADC_CS
- J5 pad 3: CH2_GND -> CH1_GND
- J5 pad 4: CH2_DAC_CS -> CH1_DAC_CS
- J5 pad 6: CH2_OUT_EN -> CH1_OUT_EN
- U2 pad 26: CTRL_CH1_ADC_CS -> CTRL_CH2_ADC_CS
- U2 pad 27: CTRL_CH1_DAC_CS -> CTRL_CH2_DAC_CS
- U2 pad 29: CTRL_CH1_OUT_EN -> CTRL_CH2_OUT_EN
- U2 pad 31: CTRL_CH2_ADC_CS -> CTRL_CH1_ADC_CS
- U2 pad 32: CTRL_CH2_DAC_CS -> CTRL_CH1_DAC_CS
- U2 pad 34: CTRL_CH2_OUT_EN -> CTRL_CH1_OUT_EN
- U3 pad 11: CH1_OUT_EN -> CH2_OUT_EN
- U3 pad 12: CH1_ADC_CS -> CH2_ADC_CS
- U3 pad 13: CH1_DAC_CS -> CH2_DAC_CS
- U3 pad 4: CTRL_CH1_ADC_CS -> CTRL_CH2_ADC_CS
- U3 pad 5: CTRL_CH1_DAC_CS -> CTRL_CH2_DAC_CS
- U3 pad 6: CTRL_CH1_OUT_EN -> CTRL_CH2_OUT_EN
- U3 pad 9: CH1_GND -> CH2_GND
- U4 pad 11: CH2_OUT_EN -> CH1_OUT_EN
- U4 pad 12: CH2_ADC_CS -> CH1_ADC_CS
- U4 pad 13: CH2_DAC_CS -> CH1_DAC_CS
- U4 pad 4: CTRL_CH2_ADC_CS -> CTRL_CH1_ADC_CS
- U4 pad 5: CTRL_CH2_DAC_CS -> CTRL_CH1_DAC_CS
- U4 pad 6: CTRL_CH2_OUT_EN -> CTRL_CH1_OUT_EN
- U4 pad 9: CH2_GND -> CH1_GND
Routing:
- net CTRL_CH2_ADC_CS: track 37.3 -> 52.0 mm
- net CTRL_CH1_ADC_CS: track 52.0 -> 37.3 mm
- net CTRL_CH2_DAC_CS: track 35.2 -> 47.8 mm
- net CTRL_CH1_DAC_CS: track 47.8 -> 35.2 mm
- net CTRL_CH2_OUT_EN: track 29.2 -> 41.1 mm
- net CTRL_CH1_OUT_EN: track 41.1 -> 29.2 mm
- net Net-(D2-K): track 42.4 -> 34.8 mm
- net CH1_GND: track 11.5 -> 18.3 mm, vias 1 -> 2
- net CH1_ADC_CS: track 14.0 -> 20.1 mm
- net CH1_DAC_CS: track 11.9 -> 17.8 mm
- net Net-(D4-K): track 24.8 -> 30.7 mm
- net CH1_OUT_EN: track 11.3 -> 15.8 mm
- net Net-(J5-Pin_9): track 6.58 -> 10.4 mm
- net Net-(J5-Pin_5): track 7.31 -> 10.5 mm
- net Net-(D2-A): track 40.6 -> 43.1 mm, vias 0 -> 1
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Other:
- board text added: "+"
- board text added: "-"
- board text added: "CH1"
- board text added: "CH2"
- board text added: "GND"
- board text added: "GPB4"
- board text added: "GPB5"
- board text added: "GPB6"
- board text added: "GPB7"
- board text added: "bench psu control v. 1.1"
- board text removed: "bench psu control v. 1.0"
